Commit message: update depth_camera

File: env/assets/urdf/ball.urdf (robot description, URDF)
Before this commit: robot ball, 1 links, 0 joints
Links:
- link ball: mass 0.5 -> 0.0008; geometry collision sphere radius=0.03; visual sphere radius=0.03

File: env/assets/urdf/box.urdf (robot description, URDF)
Before this commit: robot object, 1 links, 0 joints
Links:
- link object: mass 0.5 -> 0.1; geometry collision box size=0.06 0.04 0.008; visual box size=0.06 0.04 0.008
