Commit message: update RealmanGraspSingleObject Task

File: env/assets/urdf/box.urdf (robot description, URDF)
Before this commit: robot object, 1 links, 0 joints
Links:
- link object: mass 0.1 -> 0.116; geometry collision box size=0.234 0.046 0.05; visual box size=0.234 0.046 0.05

Commit message: fixed Grasp_dexterous_object_reward

File: env/assets/urdf/box.urdf (robot description, URDF)
Before this commit: robot object, 1 links, 0 joints
Links:
- link object: mass 0.116 -> 0.1; geometry collision box size=0.06 0.04 0.008; visual box size=0.06 0.04 0.008
