Commit message: fixed RealmanGraspSingleObecjt Task

File: env/assets/urdf/Embodied lifting robot_two wheels_RM75-B-V/urdf/Embodied lifting robot_two wheels_RM75-B-V.urdf (robot description, URDF)
Before this commit: robot Embodied lifting robot_two wheels_RM75-B-V, 37 links, 36 joints
Links:
- removed link Left_1_Link
- removed link Left_2_Link
- removed link Left_Support_Link
- removed link Right_1_Link
- removed link Right_2_Link
- removed link Right_Support_Link
- removed link hand_base
- removed link link_left_0
- removed link link_left_1
- removed link link_left_2
- removed link link_left_3
- removed link link_left_4
- removed link link_left_5
- removed link link_left_6
- removed link link_left_7
- removed link link_left_camera
- removed link link_mid_1
- removed link link_mid_2
- removed link link_mid_camera
- removed link link_right_camera
Joints:
- removed joint Left_1_Joint
- removed joint Left_2_Joint
- removed joint Left_Support_Joint
- removed joint Right_1_Joint
- removed joint Right_2_Joint
- removed joint Right_Support_Joint
- removed joint joint_hand_base
- removed joint joint_left_0
- removed joint joint_left_1
- removed joint joint_left_2
- removed joint joint_left_3
- removed joint joint_left_4
- removed joint joint_left_5
- removed joint joint_left_6
- removed joint joint_left_7
- removed joint joint_left_camera
- removed joint joint_mid_1
- removed joint joint_mid_2
- removed joint joint_mid_camera
- removed joint joint_right_camera
- joint joint_5: limit lower=-1 upper=0 effort=250 velocity=0.2 -> lower=-0.75 upper=-0.75 effort=0 velocity=0.001

File: env/assets/urdf/oreo.urdf (robot description, URDF)
Before this commit: robot object, 1 links, 0 joints
Links:
- link object: geometry collision box size=0.21 0.05 0.05; visual box size=0.21 0.05 0.05

Commit message: Single-Object Grasping Pipeline Established

File: env/assets/urdf/Embodied lifting robot_two wheels_RM75-B-V/urdf/Embodied lifting robot_two wheels_RM75-B-V.urdf (robot description, URDF)
Before this commit: robot Embodied lifting robot_two wheels_RM75-B-V, 17 links, 16 joints
Joints:
- joint joint_5: limit lower=-0.75 upper=-0.75 effort=0 velocity=0.001 -> lower=-0.9 upper=-0.9 effort=0 velocity=0.001
- joint joint_hand_base2: origin xyz=0 0 0.0228 rpy=0 0 0 -> xyz=0 0 0.0228 rpy=0 0 -1.57

File: env/assets/urdf/box.urdf (robot description, URDF)
Before this commit: robot object, 1 links, 0 joints
Links:
- link object: mass 0.1 -> 0.2; geometry collision box size=0.105 0.06 0.04; visual box size=0.105 0.06 0.04

Commit message: rewrite gym_structure and update collect traj

File: env/assets/urdf/Embodied lifting robot_two wheels_RM75-B-V/urdf/Embodied lifting robot_two wheels_RM75-B-V.urdf (robot description, URDF)
Before this commit: robot Embodied lifting robot_two wheels_RM75-B-V, 17 links, 16 joints
Links:
- added link link_mid_1, mass 0.14; collision mesh filename=package://Embodied lifting robot_two wheels_RM75-B-V/meshes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; visual mesh filename=package://Embodied lifting robot_two wheels_RM75-B-V/meshes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
- added link link_mid_2, mass 0.37; collision mesh filename=package://Embodied lifting robot_two wheels_RM75-B-V/meshes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; visual mesh filename=package://Embodied lifting robot_two wheels_RM75-B-V/meshes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
Joints:
- added joint joint_mid_1: type fixed, parent link_5, child link_mid_1, origin xyz=0 -0.0675 0.21566 rpy=0 0 1.5708, axis 0 0 1, limit lower=-0.37 upper=-0.37 effort=7 velocity=3.14
- added joint joint_mid_2: type fixed, parent link_mid_1, child link_mid_2, origin xyz=0.02 -0.027 0.0965 rpy=0 0 0, axis 0 -1 0, limit lower=-0.65 upper=-0.65 effort=7 velocity=3.14
- joint joint_5: limit lower=-0.9 upper=-0.9 effort=0 velocity=0.001 -> lower=-0.95 upper=-0.95 effort=0 velocity=0.001
